File: SMPS_BUCK_AP6320X.kicad_sch (KiCad schematic)
At the start: 0 parts

Commit message: New layout.
Parts:
- added Cb1, Cb2, Cb3, Cb4: 10 uF, kicad_lib:Samsung_Electro-Mechanics_CL10B104JB8NNNC, symbol kicad_lib:Murata_Electronics_GRM188Z71A106KA73D
- added Cd1, Cd2, Cd3, Cd4: 100 nF, kicad_lib:Samsung_Electro-Mechanics_CL10B104JB8NNNC, symbol kicad_lib:Samsung_Electro-Mechanics_CL10B104JB8NNNC
- added D1: LTST-C190KFKT, kicad_lib:Lite-On_LTST-C190KFKT, symbol kicad_lib:Lite-On_LTST-C190KFKT
- added J1: 61300411121, kicad_lib:Würth_Elektronik_61300411121, symbol kicad_lib:Würth_Elektronik_61300411121
- added L1: Abracon LLC ASPI-4030S-6R8M-T, kicad_lib:Abracon_LLC_ASPI-4030S-6R8M-T, symbol kicad_lib:Abracon_LLC_ASPI-4030S-6R8M-T
- added R1, R2, R3, R4: 10 kΩ, kicad_lib:YAGEO_RC0603FR-070RL, symbol kicad_lib:YAGEO_RC0603FR-0710KL
- added U2: AP63205WU-7, kicad_lib:TSOT23-6, symbol kicad_lib:Diodes_Incorporated_AP63205WU-7
Connections:
- new net: D1.A, R3.1
- new net: Cd1.2, L1.1, U2.5 (SW)
- new net: Cd1.1, U2.6 (BST)
- new net EN: J1.1, R4.1, U2.2 (EN)
- new net FB: Cd4.1, R1.1, R2.2, U2.1 (FB)
- new net GND: Cb1.1, Cb2.1, Cb3.1, Cb4.1, Cd2.1, Cd3.1, D1.K, J1.3, R2.1, U2.4 (GND)
- new net VIN: Cb1.2, Cd2.2, J1.2, R4.2, U2.3 (VIN)
- new net VOUT: Cb2.2, Cb3.2, Cb4.2, Cd3.2, Cd4.2, J1.4, L1.2, R1.2, R3.2

Commit message: New layout.
Parts:
- removed Cb1: 10 uF, kicad_lib:Samsung_Electro-Mechanics_CL10B104JB8NNNC, symbol kicad_lib:Murata_Electronics_GRM188Z71A106KA73D
- removed R1, R3: 10 kΩ, kicad_lib:YAGEO_RC0603FR-070RL, symbol kicad_lib:YAGEO_RC0603FR-0710KL
- added C1: 10 uF, kicad_lib:Samsung_Electro-Mechanics_CL10B104JB8NNNC, symbol kicad_lib:Murata_Electronics_GRM188R6YA106MA73D
- added C2: 1 uF, kicad_lib:Samsung_Electro-Mechanics_CL10B104JB8NNNC, symbol kicad_lib:Samsung_Electro-Mechanics_CL10A105KB8NNNC
- added R1: 0 Ω, kicad_lib:YAGEO_RC0603FR-070RL, symbol kicad_lib:YAGEO_RC0603FR-070RL
- added R3: 1 kΩ, kicad_lib:YAGEO_RC0603FR-070RL, symbol kicad_lib:YAGEO_RC0603FR-071KL
- R2: now not fitted
- renumbered U2 to U1
Connections:
- net FB: now also R1.1
- net GND: now also C1.1, C2.1
- net VIN: now also C1.2, C2.2
- net VOUT: now also R1.2, R3.1
- net at D1.A: now also R3.2
Other:
- moved on the sheet: Cb2, Cb3, Cb4, Cd1, Cd2, Cd3, Cd4, D1, J1, L1, R4, U1

Commit message: Changed inductor and layout.
Parts:
- removed Cb4: 10 uF, kicad_lib:Samsung_Electro-Mechanics_CL10B104JB8NNNC, symbol kicad_lib:Murata_Electronics_GRM188Z71A106KA73D
- removed L1: Abracon LLC ASPI-4030S-6R8M-T, kicad_lib:Abracon_LLC_ASPI-4030S-6R8M-T, symbol kicad_lib:Abracon_LLC_ASPI-4030S-6R8M-T
- added Cb3: 10 uF, kicad_lib:Samsung_Electro-Mechanics_CL10B104JB8NNNC, symbol kicad_lib:Murata_Electronics_GRM188Z71A106KA73D
- added Cf1: 100 pF, kicad_lib:Samsung_Electro-Mechanics_CL10B104JB8NNNC, symbol kicad_lib:Samsung_Electro-Mechanics_CL10C101JB8NNNC
- added L1: Abracon LLC ASPI-0628-6R8M-T1, kicad_lib:Abracon_LLC_ASPI-0628-6R8M-T1, symbol kicad_lib:Abracon_LLC_ASPI-0628-6R8M-T1
- renumbered C1 to Ca1, Cb2 to Cb1, Cb3 to Cb2, C2 to Ce1
Connections:
- net EN: now also J1.3; no longer J1.1
- net FB: now also Cf1.1; no longer Cd4.1
- net GND: now also Cd4.1, J1.2, Cb3.1; no longer J1.3
- net VIN: now also J1.1; no longer J1.2
- net VOUT: now also Cb3.2, Cf1.2, L1.2
- net at Cd1.2, U1.5 (SW): now also L1.1
Other:
- title: (none) -> AP6320X BUCK SMPS
- moved on the sheet: Ca1, Cb1, Cb2, Cd1, Cd2, Cd3, Ce1, D1, J1, R1, R2, R3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
