File: Hardware/SMPS_BUCK_AP6320X.kicad_sch (KiCad schematic)
At the start: 18 parts, among them J1 61300411121, U1 AP63205WU-7

Commit message: Added BOM files, 3D and unit prices to BOM.
Parts:
- removed L1: Abracon LLC ASPI-0628-6R8M-T1, kicad_lib:Abracon_LLC_ASPI-0628-6R8M-T1, symbol kicad_lib:Abracon_LLC_ASPI-0628-6R8M-T1
- added L1: Abracon LLC ASPI-6045S-6R8M-T, kicad_lib:Abracon_LLC_ASPI-6045S-6R8M-T, symbol kicad_lib:Abracon_LLC_ASPI-6045S-6R8M-T
- Ca1, Cf1, R1, R2, R3, R4: RoHS (none) -> Compliant; Unity Price (DigiKey, US$) (none) -> 0.1
- Cb1, Cb2, Cb3: MPN (none) -> GRM188Z71A106KA73D; Manufacturer Part Number GRM188Z71A106KA73D -> (none); RoHS (none) -> Compliant; Unity Price (DigiKey, US$) (none) -> 0.1
- Cd1, Cd2, Cd3, Cd4: MPN (none) -> CL10B104JB8NNNC; Manufacturer Part Number CL10B104JB8NNNC -> (none); RoHS (none) -> Compliant; Unity Price (DigiKey, US$) (none) -> 0.1
- Ce1: RoHS (none) -> Compliant; Unity Price (DigiKey, US$) (none) -> 0.11
- D1: RoHS (none) -> Compliant; Unity Price (DigiKey, US$) (none) -> 0.12
- J1: DigiKey (none) -> https://www.digikey.com/en/products/detail/w%C3%BCrth-elekt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; Mouser (none) -> https://www.mouser.com/ProductDetail/Wurth-Elektronik/61300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; RoHS (none) -> Compliant; Unity Price (DigiKey, US$) (none) -> 0.19; now not fitted
- U1: RoHS (none) -> Compliant; Unity Price (DigiKey, US$) (none) -> 0.8
Connections:
- net VOUT: now also L1.2
- net at Cd1.2, U1.5 (SW): now also L1.1
Other:
- note added: "CONNECTOR"
- note added: "NOTES"
- note added: "TRANSCEIVER"
- title: AP6320X BUCK SMPS -> ${TITLE}
